Commit message: Major update: Switch to +Y workspace, sparse reward, separate launch files
Changes:
- URDF: Flipped Joint 2,3,5 axes for +Y workspace
- Workspace: Y bounds changed from [-0.30,-0.15] to [+0.15,+0.30]
- World/Models: Updated target sphere and drawing_surface to +Y
- Reward: Switched to sparse (0/-1) like GitHub project
- Training: Higher LR (actor:0.001, critic:0.002), 64 opt steps
- Launch: Separated reaching (rl_training) and drawing (drawing_training)
- FK: Updated fk_ik_utils.py with flipped joint axes + debug logging
- Threshold: Tightened from 1cm to 0.75cm
- Added Neural IK, Analytical IK, PID controller, Drawing modules

File: ros2_ws/src/robot_arm2/urdf/New.xacro (robot description, xacro)
@@ -185,5 +185,5 @@
   <parent link="Link1_1"/>
   <child link="Link2_1"/>
-  <axis xyz="1.0 0.0 0.0"/>
+  <axis xyz="-1.0 0.0 0.0"/>
   <limit effort="100" velocity="100"/>
 </joint>
@@ -199,5 +199,5 @@
   <parent link="Link4_1"/>
   <child link="Link5_1"/>
-  <axis xyz="-1.0 0.0 0.0"/>
+  <axis xyz="1.0 0.0 0.0"/>
   <limit effort="100" velocity="100"/>
 </joint>
@@ -213,5 +213,5 @@
   <parent link="Link2_1"/>
   <child link="Link3_1"/>
-  <axis xyz="-1.0 0.0 0.0"/>
+  <axis xyz="1.0 0.0 0.0"/>
   <limit effort="100" velocity="100"/>
 </joint>

Commit message: feat: +Y workspace, kaymen99 hyperparams (TAU=0.05, HER reward=0)
- Fixed all files for +Y workspace (Y: 0.15 to 0.30)
- Updated neural_ik.py pos_min/max for +Y
- Updated drawing_environment.py obs bounds
- Updated deploy_on_pi.py workspace and default target
- Updated rl_environment.py workspace comments
- Changed TAU from 0.005 to 0.05 (kaymen99 style)
- Changed HER success_reward from +10 to 0 (sparse)
- Fixed episode_steps bug in train_robot.py
- Joint 4 changed to continuous in New.xacro

File: ros2_ws/src/robot_arm2/urdf/New.xacro (robot description, xacro)
@@ -188,10 +188,10 @@
   <limit effort="100" velocity="100"/>
 </joint>
-<joint name="Joint 4" type="revolute">
+<joint name="Joint 4" type="continuous">
   <origin xyz="0.032204 0.031535 0.062164" rpy="0 0 0"/>
   <parent link="Link3_1"/>
   <child link="Link4_1"/>
   <axis xyz="0.0 -1.0 0.0"/>
-  <limit upper="1.570796" lower="-1.570796" effort="100" velocity="100"/>
+  <limit effort="100" velocity="100"/>
 </joint>
 <joint name="Joint 5" type="continuous">
